Commit message: Add ros2_control

File: ros2_control_course/unit5/diffbot_description/robots/diffbot.ros2_control.xacro (robot description, xacro)
@@ -3,4 +3,27 @@
   <xacro:macro name="diffbot_ros2_control" params="name prefix use_fake_hardware:=^|false fake_sensor_commands:=^|false use_sim:=^|false">
     <!-- Add the ros2_control XML tags below this line -->
+ <ros2_control name="diff_drive" type="system">
+      <hardware>
+          <plugin>gazebo_ros2_control/GazeboSystem</plugin>
+      </hardware>
+      <joint name="left_wheel_joint">
+        <command_interface name="velocity">
+          <param name="min">-1</param>
+          <param name="max">1</param>
+        </command_interface>
+        <state_interface name="position"/>
+        <state_interface name="velocity"/>
+        <state_interface name="effort"/>
+      </joint>
+      <joint name="right_wheel_joint">
+        <command_interface name="velocity">
+          <param name="min">-1</param>
+          <param name="max">1</param>
+        </command_interface>
+        <state_interface name="position"/>
+        <state_interface name="velocity"/>
+        <state_interface name="effort"/>
+      </joint>
+    </ros2_control>
   <!-- Add the ros2_control XML tags above this line -->
   </xacro:macro>
